Commit message: begin color val ik to red for visualization purposes

File: val_viz/robot_urdf/valkyrie_A_red.urdf (robot description, URDF)
Before this commit: robot valkyrie, 69 links, 68 joints
Links:
- link torso: geometry collision mesh filename=package://val_desc/model/meshes/torso/torso_red.dae; visual mesh filename=package://val_desc/model/meshes/torso/torso_red.dae
- link torsoPitchLink: geometry collision mesh filename=package://val_desc/model/meshes/torso/torsopitch_red.dae; visual mesh filename=package://val_desc/model/meshes/torso/torsopitch_red.dae

Commit message: further red mesh color valkryie

File: val_viz/robot_urdf/valkyrie_A_red.urdf (robot description, URDF)
Before this commit: robot valkyrie, 69 links, 68 joints
Links:
- link leftElbowPitchLink: geometry collision mesh filename=package://val_desc/model/meshes/arms/aj4_left_red.dae; visual mesh filename=package://val_desc/model/meshes/arms/aj4_left_red.dae
- link leftForearmLink: geometry collision mesh filename=package://val_desc/model/meshes/arms/aj5_left_red.dae; visual mesh filename=package://val_desc/model/meshes/arms/aj5_left_red.dae
- link leftHipRollLink: geometry collision mesh filename=package://val_desc/model/meshes/legs/lj2_left_red.dae; visual mesh filename=package://val_desc/model/meshes/legs/lj2_left_red.dae
- link leftHipYawLink: geometry collision mesh filename=package://val_desc/model/meshes/legs/lj1_left_red.dae; visual mesh filename=package://val_desc/model/meshes/legs/lj1_left_red.dae
- link leftPalm: geometry collision mesh filename=package://val_desc/model/meshes/arms/palm_left_red.dae; visual mesh filename=package://val_desc/model/meshes/arms/palm_left_red.dae
- link leftShoulderPitchLink: geometry collision mesh filename=package://val_desc/model/meshes/arms/aj1_left_red.dae; visual mesh filename=package://val_desc/model/meshes/arms/aj1_left_red.dae
- link leftShoulderRollLink: geometry collision mesh filename=package://val_desc/model/meshes/arms/aj2_left_red.dae; visual mesh filename=package://val_desc/model/meshes/arms/aj2_left_red.dae
- link leftShoulderYawLink: geometry collision mesh filename=package://val_desc/model/meshes/arms/aj3_left_red.dae; visual mesh filename=package://val_desc/model/meshes/arms/aj3_left_red.dae
- link leftWristRollLink: geometry collision mesh filename=package://val_desc/model/meshes/arms/aj6_left_red.dae; visual mesh filename=package://val_desc/model/meshes/arms/aj6_left_red.dae
- link lowerNeckPitchLink: geometry collision mesh filename=package://val_desc/model/meshes/head/neckj1_red.dae; visual mesh filename=package://val_desc/model/meshes/head/neckj1_red.dae
- link neckYawLink: geometry collision mesh filename=package://val_desc/model/meshes/head/neckj2_red.dae; visual mesh filename=package://val_desc/model/meshes/head/neckj2_red.dae
- link pelvis: geometry collision mesh filename=package://val_desc/model/meshes/pelvis/pelvis_red.dae; visual mesh filename=package://val_desc/model/meshes/pelvis/pelvis_red.dae
- link rightElbowPitchLink: geometry collision mesh filename=package://val_desc/model/meshes/arms/aj4_right_red.dae; visual mesh filename=package://val_desc/model/meshes/arms/aj4_right_red.dae
- link rightForearmLink: geometry collision mesh filename=package://val_desc/model/meshes/arms/aj5_right_red.dae; visual mesh filename=package://val_desc/model/meshes/arms/aj5_right_red.dae
- link rightHipRollLink: geometry collision mesh filename=package://val_desc/model/meshes/legs/lj2_right_red.dae; visual mesh filename=package://val_desc/model/meshes/legs/lj2_right_red.dae
- link rightHipYawLink: geometry collision mesh filename=package://val_desc/model/meshes/legs/lj1_right_red.dae; visual mesh filename=package://val_desc/model/meshes/legs/lj1_right_red.dae
- link rightPalm: geometry collision mesh filename=package://val_desc/model/meshes/arms/palm_right_red.dae; visual mesh filename=package://val_desc/model/meshes/arms/palm_right_red.dae
- link rightShoulderPitchLink: geometry collision mesh filename=package://val_desc/model/meshes/arms/aj1_right_red.dae; visual mesh filename=package://val_desc/model/meshes/arms/aj1_right_red.dae
- link rightShoulderRollLink: geometry collision mesh filename=package://val_desc/model/meshes/arms/aj2_right_red.dae; visual mesh filename=package://val_desc/model/meshes/arms/aj2_right_red.dae
- link rightShoulderYawLink: geometry collision mesh filename=package://val_desc/model/meshes/arms/aj3_right_red.dae; visual mesh filename=package://val_desc/model/meshes/arms/aj3_right_red.dae
- link rightWristRollLink: geometry collision mesh filename=package://val_desc/model/meshes/arms/aj6_right_red.dae; visual mesh filename=package://val_desc/model/meshes/arms/aj6_right_red.dae
- link torsoYawLink: geometry collision mesh filename=package://val_desc/model/meshes/torso/torsoyaw_red.dae; visual mesh filename=package://val_desc/model/meshes/torso/torsoyaw_red.dae
